File: electronics/boatElectronics.kicad_sch (KiCad schematic)
At the start: 0 parts

Commit message: initial programming and schematic start
Other:
- title: Boat System Electronics -> PIC32 Boat Electronics
Changed lines of the file:
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@@
 	(paper "B")
 	(title_block
-		(title "Boat System Electronics")
+		(title "PIC32 Boat Electronics")
 		(rev "0.1")
 		(company "Ege Turan")
@@
 		)
 		(fill
-			(color 199 229 255 1.0000)
+			(color 0 0 0 0.0000)
 		)
 		(property "Sheetname" "Boat"
@@
 		)
 		(fill
-			(color 204 255 220 1.0000)
+			(color 0 0 0 0.0000)
 		)
 		(property "Sheetname" "Controller"

Commit message: cleaned code and folder structure, previous commit bug still remains
Other:
- title: PIC32 Boat Electronics -> Boat System Electronics
Changed lines of the file:
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@@
 	(paper "B")
 	(title_block
-		(title "PIC32 Boat Electronics")
+		(title "Boat System Electronics")
 		(rev "0.1")
 		(company "Ege Turan")
@@
 		)
 		(fill
-			(color 0 0 0 0.0000)
+			(color 199 229 255 1.0000)
 		)
 		(property "Sheetname" "Boat"
@@
 		)
 		(fill
-			(color 0 0 0 0.0000)
+			(color 204 255 220 1.0000)
 		)
 		(property "Sheetname" "Controller"
