File: electronics/controller.kicad_sch (KiCad schematic)
At the start: 23 parts, among them J4 UART1, M2 SG90 9g Micro Servo, SW2 Reset, SW7 SW_SPDT_LIMIT, U3 PIC32MX170F256B, U4 XBee_SMT, U5 Joystick_2_Axis_1SW

Commit message: update schematic for documentation
Parts:
- gave numbers to parts that had none: 1
Changed lines of the file:
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@@
 		(dnp no)
 		(fields_autoplaced yes)
-		(property "Reference" "U?"
+		(property "Reference" "U6"
 			(at 193.04 168.9099 0)
 			(effects
@@
 			(project "boatElectronics"
 				(path "/bd24c4db-4e36-4117-bd4f-5228ef241da9/ebf9c9fd-19f1-445b-9c7b-2cb236965a45"
-					(reference "U?")
+					(reference "U6")
 					(unit 1)
 				)
